File: Linux-capable-PCB-KiCAD/A33_GPIO.sch (KiCad schematic (older format))
At the start: 44 parts, among them J1 UART_CONN, J2 GPIO_CONN, J3 USB_A, J4 USB_A, J5 Micro_SD_Card_Det, J6 MIC_DIFF_IN, Q1 Q_PMOS_GSD, Q2 BC547, U1 A33, U2 MMA8425Q_Gsensor, U3 SRV05-4, U4 MIPI_DSI_Raspberry, U5 SRV05-4, U6 SRV05-4, Y1 24MHz, Y2 32.768kHz

Commit message: Assigned footprints to components, antenna and a couple of other footprints need to be assigned
Parts:
- C26, C27, C28, C29, C30, C31, C32, C33, C34, C35, C36, C37, C38, C39, C40: footprint (none) -> Capacitor_SMD:C_0603_1608Metric
- J1: footprint (none) -> Connector_PinHeader_2.54mm:PinHeader_1x03_P2.54mm_Vertical
- J2: footprint (none) -> Connector_PinHeader_2.54mm:PinHeader_1x10_P2.54mm_Vertical
- J3, J4: footprint (none) -> Connector_USB:USB_Micro-B_Molex-105017-0001
- J5: footprint (none) -> Connector_Card:microSD_HC_Molex_104031-0811
- J6: footprint (none) -> Connector_PinSocket_2.54mm:PinSocket_1x03_P2.54mm_Vertical
- R10, R11, R12, R13, R14, R15, R16, R17, R7, R8, R9: footprint (none) -> Resistor_SMD:R_0603_1608Metric
- TP1: footprint (none) -> TestPoint:TestPoint_Pad_1.0x1.0mm
- U1: footprint Allwinner_Technology_Co.,_Ltd.-A33-* -> eec:Allwinner_Technology_Co.,_Ltd.-A33-0
- U2: footprint (none) -> Package_DFN_QFN:QFN-16-1EP_3x3mm_P0.5mm_EP1.9x1.9mm
- U4: footprint (none) -> Connector_FFC-FPC:Molex_502244-1530_1x15-1MP_P0.5mm_Horizontal
- Y1, Y2: footprint (none) -> Crystal:Crystal_SMD_EuroQuartz_MJ-4Pin_5.0x3.2mm
Changed lines of the file:
@@
 F 0 "U1" H 1700 1265 50  0000 C CNN
 F 1 "A33" H 1700 1174 50  0000 C CNN
-F 2 "Allwinner_Technology_Co.,_Ltd.-A33-*" H 1150 1400 50  0001 L CNN
+F 2 "eec:Allwinner_Technology_Co.,_Ltd.-A33-0" H 1150 1400 50  0001 L CNN
 F 3 "http://dl.linux-sunxi.org/A33/A33_Datasheet_release1.0.pdf" H 1150 1500 50  0001 L CNN
 F 4 "1.8V ~ 3.3V" H 1150 1600 50  0001 L CNN "DC Supply Voltage for I/O"
@@
 F 0 "J5" H 10100 2317 50  0000 C CNN
 F 1 "Micro_SD_Card_Det" H 10100 2226 50  0000 C CNN
-F 2 "" H 12200 2200 50  0001 C CNN
+F 2 "Connector_Card:microSD_HC_Molex_104031-0811" H 12200 2200 50  0001 C CNN
 F 3 "https://www.hirose.com/product/en/download_file/key_name/DM3/category/Catalog/doc_file_id/49662/?file_category_id=4&item_id=195&is_series=1" H 10150 1600 50  0001 C CNN
 	1    10150 1500
@@
 F 0 "R11" V 8650 950 50  0000 C CNN
 F 1 "100k" V 8600 1100 50  0000 C CNN
-F 2 "" V 8530 1100 50  0001 C CNN
+F 2 "Resistor_SMD:R_0603_1608Metric" V 8530 1100 50  0001 C CNN
 F 3 "" H 8600 1100 50  0001 C CNN
 	1    8600 1100
@@
 F 0 "R12" V 8650 1050 50  0000 C CNN
 F 1 "100k" V 8600 1200 50  0000 C CNN
-F 2 "" V 8530 1200 50  0001 C CNN
+F 2 "Resistor_SMD:R_0603_1608Metric" V 8530 1200 50  0001 C CNN
 F 3 "" H 8600 1200 50  0001 C CNN
 	1    8600 1200
@@
 F 0 "R13" V 8650 1150 50  0000 C CNN
 F 1 "10k" V 8600 1300 50  0000 C CNN
-F 2 "" V 8530 1300 50  0001 C CNN
+F 2 "Resistor_SMD:R_0603_1608Metric" V 8530 1300 50  0001 C CNN
 F 3 "" H 8600 1300 50  0001 C CNN
 	1    8600 1300
@@
 F 0 "R16" V 8650 1750 50  0000 C CNN
 F 1 "100k" V 8600 1900 50  0000 C CNN
-F 2 "" V 8530 1900 50  0001 C CNN
+F 2 "Resistor_SMD:R_0603_1608Metric" V 8530 1900 50  0001 C CNN
 F 3 "" H 8600 1900 50  0001 C CNN
 	1    8600 1900
@@
 F 0 "R15" V 8650 1650 50  0000 C CNN
 F 1 "100k" V 8600 1800 50  0000 C CNN
-F 2 "" V 8530 1800 50  0001 C CNN
+F 2 "Resistor_SMD:R_0603_1608Metric" V 8530 1800 50  0001 C CNN
 F 3 "" H 8600 1800 50  0001 C CNN
 	1    8600 1800
@@
 F 0 "R14" V 8650 1550 50  0000 C CNN
 F 1 "100k" V 8600 1700 50  0000 C CNN
-F 2 "" V 8530 1700 50  0001 C CNN
+F 2 "Resistor_SMD:R_0603_1608Metric" V 8530 1700 50  0001 C CNN
 F 3 "" H 8600 1700 50  0001 C CNN
 	1    8600 1700
@@
 F 0 "C34" H 8115 1346 50  0000 L CNN
 F 1 "22u" H 8115 1255 50  0000 L CNN
-F 2 "" H 8038 1150 50  0001 C CNN
+F 2 "Capacitor_SMD:C_0603_1608Metric" H 8038 1150 50  0001 C CNN
 F 3 "" H 8000 1300 50  0001 C CNN
 	1    8000 1300
@@
 F 0 "C33" H 7665 1346 50  0000 L CNN
 F 1 "100n" H 7665 1255 50  0000 L CNN
-F 2 "" H 7588 1150 50  0001 C CNN
+F 2 "Capacitor_SMD:C_0603_1608Metric" H 7588 1150 50  0001 C CNN
 F 3 "" H 7550 1300 50  0001 C CNN
 	1    7550 1300
@@
 F 0 "C37" V 10300 5550 50  0000 C CNN
 F 1 "1u" V 10300 5300 50  0000 C CNN
-F 2 "" H 10388 5300 50  0001 C CNN
+F 2 "Capacitor_SMD:C_0603_1608Metric" H 10388 5300 50  0001 C CNN
 F 3 "" H 10350 5450 50  0001 C CNN
 	1    10350 5450
@@
 F 0 "C38" V 10300 5750 50  0000 C CNN
 F 1 "10u" V 10300 5500 50  0000 C CNN
-F 2 "" H 10388 5500 50  0001 C CNN
+F 2 "Capacitor_SMD:C_0603_1608Metric" H 10388 5500 50  0001 C CNN
 F 3 "" H 10350 5650 50  0001 C CNN
 	1    10350 5650
@@
 F 0 "C39" V 10300 6050 50  0000 C CNN
 F 1 "10u" V 10300 5800 50  0000 C CNN
-F 2 "" H 10388 5800 50  0001 C CNN
+F 2 "Capacitor_SMD:C_0603_1608Metric" H 10388 5800 50  0001 C CNN
 F 3 "" H 10350 5950 50  0001 C CNN
 	1    10350 5950
@@
 F 0 "C40" V 10300 6250 50  0000 C CNN
 F 1 "100n" V 10300 6000 50  0000 C CNN
-F 2 "" H 10388 6000 50  0001 C CNN
+F 2 "Capacitor_SMD:C_0603_1608Metric" H 10388 6000 50  0001 C CNN
 F 3 "" H 10350 6150 50  0001 C CNN
 	1    10350 6150
@@
 F 0 "R17" V 10700 5575 50  0000 C CNN
 F 1 "200k" V 10750 5800 50  0000 C CNN
-F 2 "" V 10680 5800 50  0001 C CNN
+F 2 "Resistor_SMD:R_0603_1608Metric" V 10680 5800 50  0001 C CNN
 F 3 "" H 10750 5800 50  0001 C CNN
 	1    10750 5800
@@
 F 0 "J1" H 700 1300 50  0000 C CNN
 F 1 "UART_CONN" V 600 1100 50  0000 C CNN
-F 2 "" H 650 1100 50  0001 C CNN
+F 2 "Connector_PinHeader_2.54mm:PinHeader_1x03_P2.54mm_Vertical" H 650 1100 50  0001 C CNN
 F 3 "~" H 650 1100 50  0001 C CNN
 	1    650  1100
@@
 F 0 "J4" H 6007 3217 50  0000 C CNN
 F 1 "USB_A" H 6007 3126 50  0000 C CNN
-F 2 "" H 6100 2700 50  0001 C CNN
+F 2 "Connector_USB:USB_Micro-B_Molex-105017-0001" H 6100 2700 50  0001 C CNN
 F 3 "" H 6100 2700 50  0001 C CNN
 	1    5950 2750
@@
 F 0 "R7" H 6880 1554 50  0000 R CNN
 F 1 "100k" H 6880 1645 50  0000 R CNN
-F 2 "" V 6880 1600 50  0001 C CNN
+F 2 "Resistor_SMD:R_0603_1608Metric" V 6880 1600 50  0001 C CNN
 F 3 "" H 6950 1600 50  0001 C CNN
 	1    6950 1600
@@
 F 0 "C36" V 7950 5500 50  0000 C CNN
 F 1 "100n" V 7950 5250 50  0000 C CNN
-F 2 "" H 8038 5250 50  0001 C CNN
+F 2 "Capacitor_SMD:C_0603_1608Metric" H 8038 5250 50  0001 C CNN
 F 3 "" H 8000 5400 50  0001 C CNN
 	1    8000 5400
@@
 F 0 "R10" V 7650 5000 50  0000 C CNN
 F 1 "R" V 7600 5150 50  0000 C CNN
-F 2 "" V 7530 5150 50  0001 C CNN
+F 2 "Resistor_SMD:R_0603_1608Metric" V 7530 5150 50  0001 C CNN
 F 3 "" H 7600 5150 50  0001 C CNN
 	1    7600 5150
@@
 F 0 "R9" V 7550 4900 50  0000 C CNN
 F 1 "R" V 7600 5050 50  0000 C CNN
-F 2 "" V 7530 5050 50  0001 C CNN
+F 2 "Resistor_SMD:R_0603_1608Metric" V 7530 5050 50  0001 C CNN
 F 3 "" H 7600 5050 50  0001 C CNN
 	1    7600 5050
@@
 F 0 "TP1" H 6958 5518 50  0000 L CNN
 F 1 "Test_Point" H 6958 5427 50  0000 L CNN
-F 2 "" H 7100 5400 50  0001 C CNN
+F 2 "TestPoint:TestPoint_Pad_1.0x1.0mm" H 7100 5400 50  0001 C CNN
 F 3 "~" H 7100 5400 50  0001 C CNN
 	1    6900 5400
@@
 F 0 "C35" V 8050 4500 50  0000 C CNN
 F 1 "10u" V 7950 4500 50  0000 C CNN
-F 2 "" H 8038 4500 50  0001 C CNN
+F 2 "Capacitor_SMD:C_0603_1608Metric" H 8038 4500 50  0001 C CNN
 F 3 "" H 8000 4650 50  0001 C CNN
 	1    8000 4650
@@
 F 0 "Y1" V 6004 5094 50  0000 L CNN
 F 1 "24MHz" V 6000 4400 50  0000 L CNN
-F 2 "" H 6050 4850 50  0001 C CNN
+F 2 "Crystal:Crystal_SMD_EuroQuartz_MJ-4Pin_5.0x3.2mm" H 6050 4850 50  0001 C CNN
 F 3 "" H 6050 4850 50  0001 C CNN
 	1    6050 4850
@@
 F 0 "C29" V 5198 4600 50  0000 C CNN
 F 1 "30p" V 5289 4600 50  0000 C CNN
-F 2 "" H 5488 4450 50  0001 C CNN
+F 2 "Capacitor_SMD:C_0603_1608Metric" H 5488 4450 50  0001 C CNN
 F 3 "" H 5450 4600 50  0001 C CNN
 	1    5450 4600
@@
 F 0 "C30" V 5198 5150 50  0000 C CNN
 F 1 "30p" V 5289 5150 50  0000 C CNN
-F 2 "" H 5488 5000 50  0001 C CNN
+F 2 "Capacitor_SMD:C_0603_1608Metric" H 5488 5000 50  0001 C CNN
 F 3 "" H 5450 5150 50  0001 C CNN
 	1    5450 5150
@@
 F 0 "Y2" V 6804 3981 50  0000 L CNN
 F 1 "32.768kHz" V 6895 3981 50  0000 L CNN
-F 2 "" H 6850 3850 50  0001 C CNN
+F 2 "Crystal:Crystal_SMD_EuroQuartz_MJ-4Pin_5.0x3.2mm" H 6850 3850 50  0001 C CNN
 F 3 "" H 6850 3850 50  0001 C CNN
 	1    6850 3850
@@
 F 0 "R8" H 7520 3896 50  0000 L CNN
 F 1 "10M" H 7520 3805 50  0000 L CNN
-F 2 "" V 7380 3850 50  0001 C CNN
+F 2 "Resistor_SMD:R_0603_1608Metric" V 7380 3850 50  0001 C CNN
 F 3 "" H 7450 3850 50  0001 C CNN
 	1    7450 3850
@@
 F 0 "C31" V 6298 3500 50  0000 C CNN
 F 1 "10p" V 6389 3500 50  0000 C CNN
-F 2 "" H 6588 3350 50  0001 C CNN
+F 2 "Capacitor_SMD:C_0603_1608Metric" H 6588 3350 50  0001 C CNN
 F 3 "" H 6550 3500 50  0001 C CNN
 	1    6550 3500
@@
 F 0 "C32" V 6298 4200 50  0000 C CNN
 F 1 "10p" V 6389 4200 50  0000 C CNN
-F 2 "" H 6588 4050 50  0001 C CNN
+F 2 "Capacitor_SMD:C_0603_1608Metric" H 6588 4050 50  0001 C CNN
 F 3 "" H 6550 4200 50  0001 C CNN
 	1    6550 4200
@@
 F 0 "U4" H 4525 2615 50  0000 C CNN
 F 1 "MIPI_DSI_Raspberry" H 4525 2524 50  0000 C CNN
-F 2 "" H 4550 1600 50  0001 C CNN
+F 2 "Connector_FFC-FPC:Molex_502244-1530_1x15-1MP_P0.5mm_Horizontal" H 4550 1600 50  0001 C CNN
 F 3 "" H 4550 1600 50  0001 C CNN
 	1    4550 1600
@@
 F 0 "U1" H 9100 3015 50  0000 C CNN
 F 1 "A33" H 9100 2924 50  0000 C CNN
-F 2 "Allwinner_Technology_Co.,_Ltd.-A33-*" H 8200 3150 50  0001 L CNN
+F 2 "eec:Allwinner_Technology_Co.,_Ltd.-A33-0" H 8200 3150 50  0001 L CNN
 F 3 "http://dl.linux-sunxi.org/A33/A33_Datasheet_release1.0.pdf" H 8200 3250 50  0001 L CNN
 F 4 "1.8V ~ 3.3V" H 8200 3350 50  0001 L CNN "DC Supply Voltage for I/O"
@@
 F 0 "J2" H 2525 1025 50  0000 L CNN
 F 1 "GPIO_CONN" V 2725 1200 50  0000 L CNN
-F 2 "" H 2650 1600 50  0001 C CNN
+F 2 "Connector_PinHeader_2.54mm:PinHeader_1x10_P2.54mm_Vertical" H 2650 1600 50  0001 C CNN
 F 3 "~" H 2650 1600 50  0001 C CNN
 	1    2650 1600
@@
 F 0 "U2" H 3225 4775 50  0000 C CNN
 F 1 "MMA8425Q_Gsensor" V 3125 5875 50  0000 C CNN
-F 2 "" H 3375 5150 50  0001 C CNN
+F 2 "Package_DFN_QFN:QFN-16-1EP_3x3mm_P0.5mm_EP1.9x1.9mm" H 3375 5150 50  0001 C CNN
 F 3 "" H 3375 5150 50  0001 C CNN
 	1    3575 5200
@@
 F 0 "C27" H 2775 4750 50  0000 L CNN
 F 1 "C" H 2775 4600 50  0000 L CNN
-F 2 "" H 2788 4525 50  0001 C CNN
+F 2 "Capacitor_SMD:C_0603_1608Metric" H 2788 4525 50  0001 C CNN
 F 3 "~" H 2750 4675 50  0001 C CNN
 	1    2750 4675
@@
 F 0 "C26" H 2450 4750 50  0000 L CNN
 F 1 "C" H 2450 4600 50  0000 L CNN
-F 2 "" H 2463 4525 50  0001 C CNN
+F 2 "Capacitor_SMD:C_0603_1608Metric" H 2463 4525 50  0001 C CNN
 F 3 "~" H 2425 4675 50  0001 C CNN
 	1    2425 4675
@@
 F 0 "C28" H 4450 4600 50  0000 L CNN
 F 1 "C" H 4450 4450 50  0000 L CNN
-F 2 "" H 4463 4375 50  0001 C CNN
+F 2 "Capacitor_SMD:C_0603_1608Metric" H 4463 4375 50  0001 C CNN
 F 3 "~" H 4425 4525 50  0001 C CNN
 	1    4425 4525
@@
 F 0 "J3" H 5057 3217 50  0000 C CNN
 F 1 "USB_A" H 5057 3126 50  0000 C CNN
-F 2 "" H 5150 2700 50  0001 C CNN
+F 2 "Connector_USB:USB_Micro-B_Molex-105017-0001" H 5150 2700 50  0001 C CNN
 F 3 "" H 5150 2700 50  0001 C CNN
 	1    5000 2750
@@
 F 0 "J6" H 10625 3350 50  0000 C CNN
 F 1 "MIC_DIFF_IN" V 10525 3150 50  0000 C CNN
-F 2 "" H 10575 3150 50  0001 C CNN
+F 2 "Connector_PinSocket_2.54mm:PinSocket_1x03_P2.54mm_Vertical" H 10575 3150 50  0001 C CNN
 F 3 "~" H 10575 3150 50  0001 C CNN
 	1    10575 3150
