File: Linux-capable-PCB-KiCAD/Linux-capable-PCB-KiCAD.kicad_pcb (KiCad board)
At the start: 4 copper layers, 168 parts, among them J1 UART_CONN, J2 GPIO_CONN, J3 USB_A, J4 USB_A, J5 Micro_SD_Card_Det, J6 MIC_DIFF_IN, J7 Barrel_Jack, U1 A33, U10 TPS62130, U11 AP131-25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

Commit message: From laptop
Parts:
- U10: footprint Package_DFN_QFN:DFN-16-1EP_4x5mm_P0.5mm_EP2.44x4.34mm -> Package_DFN_QFN:QFN-16-1EP_3x3mm_P0.5mm_EP1.7x1.7mm
- moved U12 52.4 mm to (71.4, 97.3), turned to 180 degrees
- moved C81 47.5 mm to (66.1, 100.9), turned to 270 degrees
- moved R37 46.1 mm to (81.1, 100.9), turned to 180 degrees
- moved C87 45.9 mm to (73.6, 101.4), turned to 180 degrees
- moved C89 45.8 mm to (73.6, 103.2), turned to 180 degrees
- moved L4 43.4 mm to (75.9, 97.7), turned to 270 degrees
- moved R33 43.1 mm to (74.2, 93.4), turned to 270 degrees
- moved TP6 39.6 mm to (79.7, 103.9)
- moved C83 38.8 mm to (67.9, 100.9), turned to 270 degrees
- moved R31 36.2 mm to (76.7, 94.6), turned to 180 degrees
- moved C85 33.3 mm to (69.7, 93.7), turned to 180 degrees
- moved R34 32.8 mm to (72.2, 93.4), turned to 90 degrees
- moved U10 0.74 mm to (32.2, 67.6)
Routing:
- net Net-(C87-Pad1): track 0.00 -> 21.6 mm, vias 0 -> 3
- net Net-(R31-Pad2): track 0.00 -> 3.82 mm
- net Net-(C85-Pad2): track 0.00 -> 3.70 mm
- net Net-(R33-Pad2): track 0.00 -> 3.60 mm
- added copper zone on F.Cu, net +5V
- added copper zone on F.Cu, net GND
- added copper zone on F.Cu, net Net-(C87-Pad1)
- added copper zone on F.Cu, net Net-(L4-Pad1)
