File: Linux-capable-PCB-KiCAD/Linux-capable-PCB-KiCAD.sch (KiCad schematic (older format))
At the start: 36 parts, among them U1 A33

Commit message: Od kuce
Parts:
- MK1, MK2, MK3, MK4: symbol Mechanical:Mounting_Hole -> Linux-capable-PCB-KiCAD-rescue:Mounting_Hole-Mechanical
Changed lines of the file:
@@
 $EndSheet
 $Comp
-L Mechanical:Mounting_Hole MK1
+L Linux-capable-PCB-KiCAD-rescue:Mounting_Hole-Mechanical MK1
 U 1 1 631C2B6C
 P 4100 900
@@
 $EndComp
 $Comp
-L Mechanical:Mounting_Hole MK2
+L Linux-capable-PCB-KiCAD-rescue:Mounting_Hole-Mechanical MK2
 U 1 1 631C3505
 P 4100 1200
@@
 $EndComp
 $Comp
-L Mechanical:Mounting_Hole MK3
+L Linux-capable-PCB-KiCAD-rescue:Mounting_Hole-Mechanical MK3
 U 1 1 631C36AB
 P 4100 1500
@@
 $EndComp
 $Comp
-L Mechanical:Mounting_Hole MK4
+L Linux-capable-PCB-KiCAD-rescue:Mounting_Hole-Mechanical MK4
 U 1 1 631C390C
 P 4100 1800

Commit message: Revert "Od kuce"
This reverts commit 2bece482254f98a379437a0618b8cb6327aa6629.
Parts:
- MK1, MK2, MK3, MK4: symbol Linux-capable-PCB-KiCAD-rescue:Mounting_Hole-Mechanical -> Mechanical:Mounting_Hole
Changed lines of the file:
@@
 $EndSheet
 $Comp
-L Linux-capable-PCB-KiCAD-rescue:Mounting_Hole-Mechanical MK1
+L Mechanical:Mounting_Hole MK1
 U 1 1 631C2B6C
 P 4100 900
@@
 $EndComp
 $Comp
-L Linux-capable-PCB-KiCAD-rescue:Mounting_Hole-Mechanical MK2
+L Mechanical:Mounting_Hole MK2
 U 1 1 631C3505
 P 4100 1200
@@
 $EndComp
 $Comp
-L Linux-capable-PCB-KiCAD-rescue:Mounting_Hole-Mechanical MK3
+L Mechanical:Mounting_Hole MK3
 U 1 1 631C36AB
 P 4100 1500
@@
 $EndComp
 $Comp
-L Linux-capable-PCB-KiCAD-rescue:Mounting_Hole-Mechanical MK4
+L Mechanical:Mounting_Hole MK4
 U 1 1 631C390C
 P 4100 1800
