File: Linux-capable-PCB-KiCAD/PowerSupply.sch (KiCad schematic (older format))
At the start: 59 parts, among them J7 Barrel_Jack, U10 TPS62130, U11 AP131-25, U12 TPS62130, U13 TPS62130, U9 TPS62130

Commit message: Od kuce
Parts:
- C65, C66, C67, C68, C69, C70, C71, C72, C73, C74, C75, C76, C77, C78, C79, C80, C81, C82, C83, C84, C85, C86, C87, C88, C89, C90: symbol device:C -> Linux-capable-PCB-KiCAD-rescue:C-device
- J7: symbol Connector:Barrel_Jack -> Linux-capable-PCB-KiCAD-rescue:Barrel_Jack-Connector
- L2, L3, L4, L5: symbol device:L -> Linux-capable-PCB-KiCAD-rescue:L-device
- R22, R23, R24, R25, R26, R27, R28, R29, R30, R31, R32, R33, R34, R35, R36, R37, R38: symbol device:R -> Linux-capable-PCB-KiCAD-rescue:R-device
- TP2, TP3, TP4, TP5, TP6, TP7: symbol Connector:Test_Point -> Linux-capable-PCB-KiCAD-rescue:Test_Point-Connector
- U10, U12, U13, U9: symbol dc-dc:TPS62130 -> Linux-capable-PCB-KiCAD-rescue:TPS62130-dc-dc
- U11: symbol regul:AP131-25 -> Linux-capable-PCB-KiCAD-rescue:AP131-25-regul
Changed lines of the file:
@@
 $EndDescr
 $Comp
-L device:L L2
+L Linux-capable-PCB-KiCAD-rescue:L-device L2
 U 1 1 62BC413B
 P 3850 1275
@@
 $EndComp
 $Comp
-L device:C C68
+L Linux-capable-PCB-KiCAD-rescue:C-device C68
 U 1 1 62BC65CC
 P 2225 1075
@@
 $EndComp
 $Comp
-L device:C C76
+L Linux-capable-PCB-KiCAD-rescue:C-device C76
 U 1 1 62BC712D
 P 4975 1500
@@
 $EndComp
 $Comp
-L device:C C79
+L Linux-capable-PCB-KiCAD-rescue:C-device C79
 U 1 1 62BC79BD
 P 5375 1500
@@
 $EndComp
 $Comp
-L device:R R24
+L Linux-capable-PCB-KiCAD-rescue:R-device R24
 U 1 1 62BC7E36
 P 4600 1475
@@
 $EndComp
 $Comp
-L device:R R25
+L Linux-capable-PCB-KiCAD-rescue:R-device R25
 U 1 1 62BC8763
 P 4600 1875
@@
 $EndComp
 $Comp
-L device:R R29
+L Linux-capable-PCB-KiCAD-rescue:R-device R29
 U 1 1 62BCAAD8
 P 5800 1275
@@
 $EndComp
 $Comp
-L regul:AP131-25 U11
+L Linux-capable-PCB-KiCAD-rescue:AP131-25-regul U11
 U 1 1 62C1D46A
 P 4225 5175
@@
 $EndComp
 $Comp
-L device:C C74
+L Linux-capable-PCB-KiCAD-rescue:C-device C74
 U 1 1 62C1F215
 P 3500 5350
@@
 $EndComp
 $Comp
-L device:C C78
+L Linux-capable-PCB-KiCAD-rescue:C-device C78
 U 1 1 62C1F9F5
 P 5200 5350
@@
 $EndComp
 $Comp
-L device:C C75
+L Linux-capable-PCB-KiCAD-rescue:C-device C75
 U 1 1 62C203F0
 P 4750 5350
@@
 $EndComp
 $Comp
-L device:R R28
+L Linux-capable-PCB-KiCAD-rescue:R-device R28
 U 1 1 62C9F818
 P 5425 5075
@@
 	5625 5075 5625 4975
 $Comp
-L Connector:Barrel_Jack J7
+L Linux-capable-PCB-KiCAD-rescue:Barrel_Jack-Connector J7
 U 1 1 62CD6E53
 P 1325 5075
@@
 	1775 4550 1775 4850
 $Comp
-L device:C C67
+L Linux-capable-PCB-KiCAD-rescue:C-device C67
 U 1 1 62CFF74E
 P 1950 5075
@@
 	1775 5300 1775 5600
 $Comp
-L device:C C72
+L Linux-capable-PCB-KiCAD-rescue:C-device C72
 U 1 1 62D1A992
 P 2425 5075
@@
 	1950 4850 2425 4850
 $Comp
-L device:C C73
+L Linux-capable-PCB-KiCAD-rescue:C-device C73
 U 1 1 62D64A42
 P 2925 5075
@@
 Connection ~ 2425 5300
 $Comp
-L dc-dc:TPS62130 U9
+L Linux-capable-PCB-KiCAD-rescue:TPS62130-dc-dc U9
 U 1 1 62DE493B
 P 3200 1475
@@
 	4075 1275 4000 1275
 $Comp
-L device:R R22
+L Linux-capable-PCB-KiCAD-rescue:R-device R22
 U 1 1 62E0D77F
 P 4225 1425
@@
 	2225 900  2225 925
 $Comp
-L device:C C65
+L Linux-capable-PCB-KiCAD-rescue:C-device C65
 U 1 1 62F544E5
 P 1775 1075
@@
 	1775 900  2225 900
 $Comp
-L device:C C70
+L Linux-capable-PCB-KiCAD-rescue:C-device C70
 U 1 1 62F72FB4
 P 2425 1700
@@
 	6100 1275 5950 1275
 $Comp
-L device:L L3
+L Linux-capable-PCB-KiCAD-rescue:L-device L3
 U 1 1 62FEEF27
 P 3850 3175
@@
 $EndComp
 $Comp
-L device:C C69
+L Linux-capable-PCB-KiCAD-rescue:C-device C69
 U 1 1 62FEEF31
 P 2225 2975
@@
 $EndComp
 $Comp
-L device:C C77
+L Linux-capable-PCB-KiCAD-rescue:C-device C77
 U 1 1 62FEEF3B
 P 4975 3400
@@
 $EndComp
 $Comp
-L device:C C80
+L Linux-capable-PCB-KiCAD-rescue:C-device C80
 U 1 1 62FEEF45
 P 5375 3400
@@
 $EndComp
 $Comp
-L device:R R26
+L Linux-capable-PCB-KiCAD-rescue:R-device R26
 U 1 1 62FEEF4F
 P 4600 3375
@@
 $EndComp
 $Comp
-L device:R R27
+L Linux-capable-PCB-KiCAD-rescue:R-device R27
 U 1 1 62FEEF59
 P 4600 3775
@@
 $EndComp
 $Comp
-L device:R R30
+L Linux-capable-PCB-KiCAD-rescue:R-device R30
 U 1 1 62FEEF8B
 P 5800 3175
@@
 $EndComp
 $Comp
-L dc-dc:TPS62130 U10
+L Linux-capable-PCB-KiCAD-rescue:TPS62130-dc-dc U10
 U 1 1 62FEEFA9
 P 3200 3375
@@
 	4075 3175 4000 3175
 $Comp
-L device:R R23
+L Linux-capable-PCB-KiCAD-rescue:R-device R23
 U 1 1 62FEEFB7
 P 4225 3325
@@
 	2225 2800 2225 2825
 $Comp
-L device:C C66
+L Linux-capable-PCB-KiCAD-rescue:C-device C66
 U 1 1 62FEF007
 P 1775 2975
@@
 	1775 2800 2225 2800
 $Comp
-L device:C C71
+L Linux-capable-PCB-KiCAD-rescue:C-device C71
 U 1 1 62FEF01E
 P 2425 3600
@@
 $EndComp
 $Comp
-L device:L L5
+L Linux-capable-PCB-KiCAD-rescue:L-device L5
 U 1 1 63044212
 P 8600 1325
@@
 $EndComp
 $Comp
-L device:C C84
+L Linux-capable-PCB-KiCAD-rescue:C-device C84
 U 1 1 6304422E
 P 6975 1125
@@
 $EndComp
 $Comp
-L device:C C88
+L Linux-capable-PCB-KiCAD-rescue:C-device C88
 U 1 1 63044238
 P 9725 1550
@@
 $EndComp
 $Comp
-L device:C C90
+L Linux-capable-PCB-KiCAD-rescue:C-device C90
 U 1 1 63044242
 P 10125 1550
@@
 $EndComp
 $Comp
-L device:R R35
+L Linux-capable-PCB-KiCAD-rescue:R-device R35
 U 1 1 6304424C
 P 9350 1525
@@
 $EndComp
 $Comp
-L device:R R36
+L Linux-capable-PCB-KiCAD-rescue:R-device R36
 U 1 1 63044256
 P 9350 1925
@@
 $EndComp
 $Comp
-L device:R R38
+L Linux-capable-PCB-KiCAD-rescue:R-device R38
 U 1 1 63044288
 P 10550 1325
@@
 $EndComp
 $Comp
-L dc-dc:TPS62130 U13
+L Linux-capable-PCB-KiCAD-rescue:TPS62130-dc-dc U13
 U 1 1 630442A6
 P 7950 1525
@@
 	8825 1325 8750 1325
 $Comp
-L device:R R32
+L Linux-capable-PCB-KiCAD-rescue:R-device R32
 U 1 1 630442B4
 P 8975 1475
@@
 	6975 950  6975 975
 $Comp
-L device:C C82
+L Linux-capable-PCB-KiCAD-rescue:C-device C82
 U 1 1 63044304
 P 6525 1125
@@
 	6525 950  6975 950
 $Comp
-L device:C C86
+L Linux-capable-PCB-KiCAD-rescue:C-device C86
 U 1 1 6304431B
 P 7175 1750
@@
 	10850 1325 10700 1325
 $Comp
-L device:L L4
+L Linux-capable-PCB-KiCAD-rescue:L-device L4
 U 1 1 630969E4
 P 8525 3225
@@
 $EndComp
 $Comp
-L device:C C83
+L Linux-capable-PCB-KiCAD-rescue:C-device C83
 U 1 1 63096A00
 P 6900 3025
@@
 $EndComp
 $Comp
-L device:C C87
+L Linux-capable-PCB-KiCAD-rescue:C-device C87
 U 1 1 63096A0A
 P 9650 3450
@@
 $EndComp
 $Comp
-L device:C C89
+L Linux-capable-PCB-KiCAD-rescue:C-device C89
 U 1 1 63096A14
 P 10050 3450
@@
 $EndComp
 $Comp
-L device:R R33
+L Linux-capable-PCB-KiCAD-rescue:R-device R33
 U 1 1 63096A1E
 P 9275 3425
@@
 $EndComp
 $Comp
-L device:R R34
+L Linux-capable-PCB-KiCAD-rescue:R-device R34
 U 1 1 63096A28
 P 9275 3825
@@
 $EndComp
 $Comp
-L device:R R37
+L Linux-capable-PCB-KiCAD-rescue:R-device R37
 U 1 1 63096A5A
 P 10475 3225
@@
 $EndComp
 $Comp
-L dc-dc:TPS62130 U12
+L Linux-capable-PCB-KiCAD-rescue:TPS62130-dc-dc U12
 U 1 1 63096A6E
 P 7875 3425
@@
 	8750 3225 8675 3225
 $Comp
-L device:R R31
+L Linux-capable-PCB-KiCAD-rescue:R-device R31
 U 1 1 63096A7C
 P 8900 3375
@@
 	6900 2850 6900 2875
 $Comp
-L device:C C81
+L Linux-capable-PCB-KiCAD-rescue:C-device C81
 U 1 1 63096ACC
 P 6450 3025
@@
 	6450 2850 6900 2850
 $Comp
-L device:C C85
+L Linux-capable-PCB-KiCAD-rescue:C-device C85
 U 1 1 63096AE3
 P 7100 3650
@@
 	7875 4025 7875 4075
 $Comp
-L Connector:Test_Point TP4
+L Linux-capable-PCB-KiCAD-rescue:Test_Point-Connector TP4
 U 1 1 6317DC3B
 P 5375 950
@@
 	5375 950  5375 1275
 $Comp
-L Connector:Test_Point TP7
+L Linux-capable-PCB-KiCAD-rescue:Test_Point-Connector TP7
 U 1 1 6318B766
 P 10125 1000
@@
 	10125 1000 10125 1325
 $Comp
-L Connector:Test_Point TP6
+L Linux-capable-PCB-KiCAD-rescue:Test_Point-Connector TP6
 U 1 1 63198008
 P 10050 2900
@@
 	10050 2900 10050 3225
 $Comp
-L Connector:Test_Point TP5
+L Linux-capable-PCB-KiCAD-rescue:Test_Point-Connector TP5
 U 1 1 631A49EB
 P 5375 2850
@@
 	5375 2850 5375 3175
 $Comp
-L Connector:Test_Point TP3
+L Linux-capable-PCB-KiCAD-rescue:Test_Point-Connector TP3
 U 1 1 631B3B9B
 P 5200 4750
@@
 	5200 4750 5200 5075
 $Comp
-L Connector:Test_Point TP2
+L Linux-capable-PCB-KiCAD-rescue:Test_Point-Connector TP2
 U 1 1 631C6D49
 P 2925 4525

Commit message: Revert "Od kuce"
This reverts commit 2bece482254f98a379437a0618b8cb6327aa6629.
Parts:
- C65, C66, C67, C68, C69, C70, C71, C72, C73, C74, C75, C76, C77, C78, C79, C80, C81, C82, C83, C84, C85, C86, C87, C88, C89, C90: symbol Linux-capable-PCB-KiCAD-rescue:C-device -> device:C
- J7: symbol Linux-capable-PCB-KiCAD-rescue:Barrel_Jack-Connector -> Connector:Barrel_Jack
- L2, L3, L4, L5: symbol Linux-capable-PCB-KiCAD-rescue:L-device -> device:L
- R22, R23, R24, R25, R26, R27, R28, R29, R30, R31, R32, R33, R34, R35, R36, R37, R38: symbol Linux-capable-PCB-KiCAD-rescue:R-device -> device:R
- TP2, TP3, TP4, TP5, TP6, TP7: symbol Linux-capable-PCB-KiCAD-rescue:Test_Point-Connector -> Connector:Test_Point
- U10, U12, U13, U9: symbol Linux-capable-PCB-KiCAD-rescue:TPS62130-dc-dc -> dc-dc:TPS62130
- U11: symbol Linux-capable-PCB-KiCAD-rescue:AP131-25-regul -> regul:AP131-25
Changed lines of the file:
@@
 $EndDescr
 $Comp
-L Linux-capable-PCB-KiCAD-rescue:L-device L2
+L device:L L2
 U 1 1 62BC413B
 P 3850 1275
@@
 $EndComp
 $Comp
-L Linux-capable-PCB-KiCAD-rescue:C-device C68
+L device:C C68
 U 1 1 62BC65CC
 P 2225 1075
@@
 $EndComp
 $Comp
-L Linux-capable-PCB-KiCAD-rescue:C-device C76
+L device:C C76
 U 1 1 62BC712D
 P 4975 1500
@@
 $EndComp
 $Comp
-L Linux-capable-PCB-KiCAD-rescue:C-device C79
+L device:C C79
 U 1 1 62BC79BD
 P 5375 1500
@@
 $EndComp
 $Comp
-L Linux-capable-PCB-KiCAD-rescue:R-device R24
+L device:R R24
 U 1 1 62BC7E36
 P 4600 1475
@@
 $EndComp
 $Comp
-L Linux-capable-PCB-KiCAD-rescue:R-device R25
+L device:R R25
 U 1 1 62BC8763
 P 4600 1875
@@
 $EndComp
 $Comp
-L Linux-capable-PCB-KiCAD-rescue:R-device R29
+L device:R R29
 U 1 1 62BCAAD8
 P 5800 1275
@@
 $EndComp
 $Comp
-L Linux-capable-PCB-KiCAD-rescue:AP131-25-regul U11
+L regul:AP131-25 U11
 U 1 1 62C1D46A
 P 4225 5175
@@
 $EndComp
 $Comp
-L Linux-capable-PCB-KiCAD-rescue:C-device C74
+L device:C C74
 U 1 1 62C1F215
 P 3500 5350
@@
 $EndComp
 $Comp
-L Linux-capable-PCB-KiCAD-rescue:C-device C78
+L device:C C78
 U 1 1 62C1F9F5
 P 5200 5350
@@
 $EndComp
 $Comp
-L Linux-capable-PCB-KiCAD-rescue:C-device C75
+L device:C C75
 U 1 1 62C203F0
 P 4750 5350
@@
 $EndComp
 $Comp
-L Linux-capable-PCB-KiCAD-rescue:R-device R28
+L device:R R28
 U 1 1 62C9F818
 P 5425 5075
@@
 	5625 5075 5625 4975
 $Comp
-L Linux-capable-PCB-KiCAD-rescue:Barrel_Jack-Connector J7
+L Connector:Barrel_Jack J7
 U 1 1 62CD6E53
 P 1325 5075
@@
 	1775 4550 1775 4850
 $Comp
-L Linux-capable-PCB-KiCAD-rescue:C-device C67
+L device:C C67
 U 1 1 62CFF74E
 P 1950 5075
@@
 	1775 5300 1775 5600
 $Comp
-L Linux-capable-PCB-KiCAD-rescue:C-device C72
+L device:C C72
 U 1 1 62D1A992
 P 2425 5075
@@
 	1950 4850 2425 4850
 $Comp
-L Linux-capable-PCB-KiCAD-rescue:C-device C73
+L device:C C73
 U 1 1 62D64A42
 P 2925 5075
@@
 Connection ~ 2425 5300
 $Comp
-L Linux-capable-PCB-KiCAD-rescue:TPS62130-dc-dc U9
+L dc-dc:TPS62130 U9
 U 1 1 62DE493B
 P 3200 1475
@@
 	4075 1275 4000 1275
 $Comp
-L Linux-capable-PCB-KiCAD-rescue:R-device R22
+L device:R R22
 U 1 1 62E0D77F
 P 4225 1425
@@
 	2225 900  2225 925
 $Comp
-L Linux-capable-PCB-KiCAD-rescue:C-device C65
+L device:C C65
 U 1 1 62F544E5
 P 1775 1075
@@
 	1775 900  2225 900
 $Comp
-L Linux-capable-PCB-KiCAD-rescue:C-device C70
+L device:C C70
 U 1 1 62F72FB4
 P 2425 1700
@@
 	6100 1275 5950 1275
 $Comp
-L Linux-capable-PCB-KiCAD-rescue:L-device L3
+L device:L L3
 U 1 1 62FEEF27
 P 3850 3175
@@
 $EndComp
 $Comp
-L Linux-capable-PCB-KiCAD-rescue:C-device C69
+L device:C C69
 U 1 1 62FEEF31
 P 2225 2975
@@
 $EndComp
 $Comp
-L Linux-capable-PCB-KiCAD-rescue:C-device C77
+L device:C C77
 U 1 1 62FEEF3B
 P 4975 3400
@@
 $EndComp
 $Comp
-L Linux-capable-PCB-KiCAD-rescue:C-device C80
+L device:C C80
 U 1 1 62FEEF45
 P 5375 3400
@@
 $EndComp
 $Comp
-L Linux-capable-PCB-KiCAD-rescue:R-device R26
+L device:R R26
 U 1 1 62FEEF4F
 P 4600 3375
@@
 $EndComp
 $Comp
-L Linux-capable-PCB-KiCAD-rescue:R-device R27
+L device:R R27
 U 1 1 62FEEF59
 P 4600 3775
@@
 $EndComp
 $Comp
-L Linux-capable-PCB-KiCAD-rescue:R-device R30
+L device:R R30
 U 1 1 62FEEF8B
 P 5800 3175
@@
 $EndComp
 $Comp
-L Linux-capable-PCB-KiCAD-rescue:TPS62130-dc-dc U10
+L dc-dc:TPS62130 U10
 U 1 1 62FEEFA9
 P 3200 3375
@@
 	4075 3175 4000 3175
 $Comp
-L Linux-capable-PCB-KiCAD-rescue:R-device R23
+L device:R R23
 U 1 1 62FEEFB7
 P 4225 3325
@@
 	2225 2800 2225 2825
 $Comp
-L Linux-capable-PCB-KiCAD-rescue:C-device C66
+L device:C C66
 U 1 1 62FEF007
 P 1775 2975
@@
 	1775 2800 2225 2800
 $Comp
-L Linux-capable-PCB-KiCAD-rescue:C-device C71
+L device:C C71
 U 1 1 62FEF01E
 P 2425 3600
@@
 $EndComp
 $Comp
-L Linux-capable-PCB-KiCAD-rescue:L-device L5
+L device:L L5
 U 1 1 63044212
 P 8600 1325
@@
 $EndComp
 $Comp
-L Linux-capable-PCB-KiCAD-rescue:C-device C84
+L device:C C84
 U 1 1 6304422E
 P 6975 1125
@@
 $EndComp
 $Comp
-L Linux-capable-PCB-KiCAD-rescue:C-device C88
+L device:C C88
 U 1 1 63044238
 P 9725 1550
@@
 $EndComp
 $Comp
-L Linux-capable-PCB-KiCAD-rescue:C-device C90
+L device:C C90
 U 1 1 63044242
 P 10125 1550
@@
 $EndComp
 $Comp
-L Linux-capable-PCB-KiCAD-rescue:R-device R35
+L device:R R35
 U 1 1 6304424C
 P 9350 1525
@@
 $EndComp
 $Comp
-L Linux-capable-PCB-KiCAD-rescue:R-device R36
+L device:R R36
 U 1 1 63044256
 P 9350 1925
@@
 $EndComp
 $Comp
-L Linux-capable-PCB-KiCAD-rescue:R-device R38
+L device:R R38
 U 1 1 63044288
 P 10550 1325
@@
 $EndComp
 $Comp
-L Linux-capable-PCB-KiCAD-rescue:TPS62130-dc-dc U13
+L dc-dc:TPS62130 U13
 U 1 1 630442A6
 P 7950 1525
@@
 	8825 1325 8750 1325
 $Comp
-L Linux-capable-PCB-KiCAD-rescue:R-device R32
+L device:R R32
 U 1 1 630442B4
 P 8975 1475
@@
 	6975 950  6975 975
 $Comp
-L Linux-capable-PCB-KiCAD-rescue:C-device C82
+L device:C C82
 U 1 1 63044304
 P 6525 1125
@@
 	6525 950  6975 950
 $Comp
-L Linux-capable-PCB-KiCAD-rescue:C-device C86
+L device:C C86
 U 1 1 6304431B
 P 7175 1750
@@
 	10850 1325 10700 1325
 $Comp
-L Linux-capable-PCB-KiCAD-rescue:L-device L4
+L device:L L4
 U 1 1 630969E4
 P 8525 3225
@@
 $EndComp
 $Comp
-L Linux-capable-PCB-KiCAD-rescue:C-device C83
+L device:C C83
 U 1 1 63096A00
 P 6900 3025
@@
 $EndComp
 $Comp
-L Linux-capable-PCB-KiCAD-rescue:C-device C87
+L device:C C87
 U 1 1 63096A0A
 P 9650 3450
@@
 $EndComp
 $Comp
-L Linux-capable-PCB-KiCAD-rescue:C-device C89
+L device:C C89
 U 1 1 63096A14
 P 10050 3450
@@
 $EndComp
 $Comp
-L Linux-capable-PCB-KiCAD-rescue:R-device R33
+L device:R R33
 U 1 1 63096A1E
 P 9275 3425
@@
 $EndComp
 $Comp
-L Linux-capable-PCB-KiCAD-rescue:R-device R34
+L device:R R34
 U 1 1 63096A28
 P 9275 3825
@@
 $EndComp
 $Comp
-L Linux-capable-PCB-KiCAD-rescue:R-device R37
+L device:R R37
 U 1 1 63096A5A
 P 10475 3225
@@
 $EndComp
 $Comp
-L Linux-capable-PCB-KiCAD-rescue:TPS62130-dc-dc U12
+L dc-dc:TPS62130 U12
 U 1 1 63096A6E
 P 7875 3425
@@
 	8750 3225 8675 3225
 $Comp
-L Linux-capable-PCB-KiCAD-rescue:R-device R31
+L device:R R31
 U 1 1 63096A7C
 P 8900 3375
@@
 	6900 2850 6900 2875
 $Comp
-L Linux-capable-PCB-KiCAD-rescue:C-device C81
+L device:C C81
 U 1 1 63096ACC
 P 6450 3025
@@
 	6450 2850 6900 2850
 $Comp
-L Linux-capable-PCB-KiCAD-rescue:C-device C85
+L device:C C85
 U 1 1 63096AE3
 P 7100 3650
@@
 	7875 4025 7875 4075
 $Comp
-L Linux-capable-PCB-KiCAD-rescue:Test_Point-Connector TP4
+L Connector:Test_Point TP4
 U 1 1 6317DC3B
 P 5375 950
@@
 	5375 950  5375 1275
 $Comp
-L Linux-capable-PCB-KiCAD-rescue:Test_Point-Connector TP7
+L Connector:Test_Point TP7
 U 1 1 6318B766
 P 10125 1000
@@
 	10125 1000 10125 1325
 $Comp
-L Linux-capable-PCB-KiCAD-rescue:Test_Point-Connector TP6
+L Connector:Test_Point TP6
 U 1 1 63198008
 P 10050 2900
@@
 	10050 2900 10050 3225
 $Comp
-L Linux-capable-PCB-KiCAD-rescue:Test_Point-Connector TP5
+L Connector:Test_Point TP5
 U 1 1 631A49EB
 P 5375 2850
@@
 	5375 2850 5375 3175
 $Comp
-L Linux-capable-PCB-KiCAD-rescue:Test_Point-Connector TP3
+L Connector:Test_Point TP3
 U 1 1 631B3B9B
 P 5200 4750
@@
 	5200 4750 5200 5075
 $Comp
-L Linux-capable-PCB-KiCAD-rescue:Test_Point-Connector TP2
+L Connector:Test_Point TP2
 U 1 1 631C6D49
 P 2925 4525
