File: Linux-capable-PCB-KiCAD/PowerSupply.sch (KiCad schematic (older format))
At the start: 59 parts, among them J7 Barrel_Jack, U10 TPS62130, U11 AP131-25, U12 TPS62130, U13 TPS62130, U9 TPS62130

Commit message: Assigned footprints to components, antenna and a couple of other footprints need to be assigned
Parts:
- C65, C66, C67, C68, C69, C70, C71, C72, C73, C74, C75, C76, C77, C78, C79, C80, C81, C82, C83, C84, C85, C86, C87, C88, C89, C90: footprint (none) -> Capacitor_SMD:C_0603_1608Metric
- J7: footprint (none) -> Connector_BarrelJack:BarrelJack_CUI_PJ-063AH_Horizontal
- L2, L3, L4, L5: footprint (none) -> Inductor_SMD:L_0603_1608Metric
- R22, R23, R24, R25, R26, R27, R28, R29, R30, R31, R32, R33, R34, R35, R36, R37, R38: footprint (none) -> Resistor_SMD:R_0603_1608Metric
- TP2, TP3, TP4, TP5, TP6, TP7: footprint (none) -> TestPoint:TestPoint_Pad_1.0x1.0mm
- U10: footprint Housings_DFN_QFN:QFN-16-1EP_3x3mm_Pitch0.5mm -> Package_DFN_QFN:DFN-16-1EP_4x5mm_P0.5mm_EP2.44x4.34mm
- U11: footprint TO_SOT_Packages_SMD:SOT-23-5 -> Package_TO_SOT_SMD:SOT-23-5
- U12, U13, U9: footprint Housings_DFN_QFN:QFN-16-1EP_3x3mm_Pitch0.5mm -> Package_DFN_QFN:QFN-16-1EP_3x3mm_P0.5mm_EP1.7x1.7mm

Commit message: CPU and DDR3 connected
Connections:
- net +1V35 renamed +1V5
Other:
- note added: "FIX RESISTOR VALUES"
Changed lines of the file:
@@
 	10850 1325 10700 1325
-$Comp
-L power:+1V35 #PWR0251
-U 1 1 63061F46
-P 10850 1125
-F 0 "#PWR0251" H 10850 975 50  0001 C CNN
-F 1 "+1V35" H 10865 1298 50  0000 C CNN
-F 2 "" H 10850 1125 50  0001 C CNN
-F 3 "" H 10850 1125 50  0001 C CNN
-	1    10850 1125
-	1    0    0    -1
-$EndComp
 $Comp
 L device:L L4
@@
 	2925 4525 2925 4850
 Connection ~ 2925 4850
+$Comp
+L power:+1V5 #PWR0251
+U 1 1 62C74527
+P 10850 1125
+F 0 "#PWR0251" H 10850 975 50  0001 C CNN
+F 1 "+1V5" H 10865 1298 50  0000 C CNN
+F 2 "" H 10850 1125 50  0001 C CNN
+F 3 "" H 10850 1125 50  0001 C CNN
+	1    10850 1125
+	1    0    0    -1
+$EndComp
+Text Notes 7875 2625 0    157  ~ 0
+FIX RESISTOR VALUES
 $EndSCHEMATC

Commit message: From laptop
Parts:
- U10: footprint Package_DFN_QFN:DFN-16-1EP_4x5mm_P0.5mm_EP2.44x4.34mm -> Package_DFN_QFN:QFN-16-1EP_3x3mm_P0.5mm_EP1.7x1.7mm
Changed lines of the file:
@@
 F 0 "U10" H 2950 3825 50  0000 C CNN
 F 1 "TPS62130" H 3525 2900 50  0000 C CNN
-F 2 "Package_DFN_QFN:DFN-16-1EP_4x5mm_P0.5mm_EP2.44x4.34mm" H 3350 2925 50  0001 L CNN
+F 2 "Package_DFN_QFN:QFN-16-1EP_3x3mm_P0.5mm_EP1.7x1.7mm" H 3350 2925 50  0001 L CNN
 F 3 "http://www.ti.com/lit/ds/symlink/tps62130.pdf" H 3200 3375 50  0001 C CNN
 	1    3200 3375
