File: Linux-capable-PCB-KiCAD/Linux-capable-PCB-KiCAD.kicad_sch (KiCad schematic)
At the start: 36 parts

Commit message: Dodao 3.3V na SD karticu, treba zamjeniti SD konektor, zavrsio napjanje, treba izracunati vrijednosti otpornika i footprint preci za komponente
Parts:
- C1, C10, C11, C14, C15, C16, C18, C19, C2, C20, C21, C22, C25, C3, C4, C5, C6, C8, C9: value (none) -> 100n; footprint (none) -> Capacitor_SMD:C_0603_1608Metric
- C12, C13, C23, C24, C7: value (none) -> 22u; footprint (none) -> Capacitor_SMD:C_0603_1608Metric
- C17: value (none) -> 10u; footprint (none) -> Capacitor_SMD:C_0603_1608Metric
- MK1, MK2, MK3, MK4: value (none) -> Mounting_Hole; footprint (none) -> MountingHole:MountingHole_3mm
- R1, R2: value (none) -> 1k; footprint (none) -> Resistor_SMD:R_0603_1608Metric
- R3, R4: value (none) -> 22R; footprint (none) -> Resistor_SMD:R_0603_1608Metric
- R5: value (none) -> 240R; footprint (none) -> Resistor_SMD:R_0603_1608Metric
- R6: value (none) -> 0R; footprint (none) -> Resistor_SMD:R_0603_1608Metric
- U1: value (none) -> A33; footprint (none) -> eec:Allwinner_Technology_Co.,_Ltd.-A33-0

Commit message: message
Parts:
- removed C12: 22u, Capacitor_SMD:C_0603_1608Metric, symbol Linux-capable-PCB-KiCAD-rescue:C-device
- removed C16, C19, C4, C8: 100n, Capacitor_SMD:C_0603_1608Metric, symbol Linux-capable-PCB-KiCAD-rescue:C-device
