File: Linux-capable-PCB-KiCAD/RAM.kicad_sch (KiCad schematic)
At the start: 23 parts

Commit message: Dodao 3.3V na SD karticu, treba zamjeniti SD konektor, zavrsio napjanje, treba izracunati vrijednosti otpornika i footprint preci za komponente
Parts:
- C46, C47, C48, C49, C50, C51, C52, C53, C54, C55, C56, C57, C58, C59, C60, C61, C62, C63, C64: value (none) -> 100n; footprint (none) -> Capacitor_SMD:C_0603_1608Metric
- R19: value (none) -> 240R; footprint (none) -> Resistor_SMD:R_0603_1608Metric
- R20, R21: value (none) -> 1k 1%; footprint (none) -> Resistor_SMD:R_0603_1608Metric
- U8: value (none) -> HTQ4G63AFR-PCB; footprint (none) -> Package_BGA:BGA-96_9.0x13.0mm_Layout2x3x16_P0.8mm

Commit message: message
Parts:
- removed C50, C53: 100n, Capacitor_SMD:C_0603_1608Metric, symbol Linux-capable-PCB-KiCAD-rescue:C-Device
Changed lines of the file:
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@@
   (junction (at 262.89 68.58) (diameter 0) (color 0 0 0 0)
-  )
-  (junction (at 139.7 79.375) (diameter 0) (color 0 0 0 0)
   )
   (junction (at 35.56 76.835) (diameter 0) (color 0 0 0 0)
@@
     (stroke (width 0) (type default) (color 0 0 0 0))
   )
-  (wire (pts (xy 139.7 79.375) (xy 145.415 79.375))
-    (stroke (width 0) (type default) (color 0 0 0 0))
-  )
   (wire (pts (xy 95.25 43.815) (xy 105.41 43.815))
     (stroke (width 0) (type default) (color 0 0 0 0))
@@
     (stroke (width 0) (type default) (color 0 0 0 0))
   )
-  (wire (pts (xy 132.715 92.71) (xy 132.715 90.17))
-    (stroke (width 0) (type default) (color 0 0 0 0))
-  )
   (wire (pts (xy 206.375 108.585) (xy 206.375 106.045))
     (stroke (width 0) (type default) (color 0 0 0 0))
@@
     (stroke (width 0) (type default) (color 0 0 0 0))
   )
-  (wire (pts (xy 132.715 82.55) (xy 132.715 79.375))
-    (stroke (width 0) (type default) (color 0 0 0 0))
-  )
   (wire (pts (xy 170.18 43.815) (xy 179.07 43.815))
     (stroke (width 0) (type default) (color 0 0 0 0))
@@
     (stroke (width 0) (type default) (color 0 0 0 0))
   )
-  (wire (pts (xy 145.415 79.375) (xy 145.415 82.55))
-    (stroke (width 0) (type default) (color 0 0 0 0))
-  )
   (wire (pts (xy 262.89 93.98) (xy 262.89 96.52))
     (stroke (width 0) (type default) (color 0 0 0 0))
@@
     (stroke (width 0) (type default) (color 0 0 0 0))
   )
-  (wire (pts (xy 139.7 77.47) (xy 139.7 79.375))
-    (stroke (width 0) (type default) (color 0 0 0 0))
-  )
   (wire (pts (xy 257.175 91.44) (xy 262.89 91.44))
     (stroke (width 0) (type default) (color 0 0 0 0))
@@
     (stroke (width 0) (type default) (color 0 0 0 0))
   )
-  (wire (pts (xy 145.415 92.71) (xy 145.415 90.17))
-    (stroke (width 0) (type default) (color 0 0 0 0))
-  )
   (bus (pts (xy 80.01 85.725) (xy 77.47 83.185))
     (stroke (width 0) (type default) (color 0 0 0 0))
@@
   )
   (wire (pts (xy 262.89 91.44) (xy 262.89 93.98))
-    (stroke (width 0) (type default) (color 0 0 0 0))
-  )
-  (wire (pts (xy 132.715 79.375) (xy 139.7 79.375))
     (stroke (width 0) (type default) (color 0 0 0 0))
   )
@@
     (pin "T8")
   )
-  (symbol (lib_id "Linux-capable-PCB-KiCAD-rescue:C-Device") (at 145.415 86.36 0) (unit 1)
-    (in_bom yes) (on_board yes)
-    (property "Reference" "C53" (id 0) (at 148.336 85.1916 0)
-      (effects (font (size 1.27 1.27)) (justify left))
-    )
-    (property "Value" "100n" (id 1) (at 148.336 87.503 0)
-      (effects (font (size 1.27 1.27)) (justify left))
-    )
-    (property "Footprint" "Capacitor_SMD:C_0603_1608Metric" (id 2) (at 146.3802 90.17 0)
-      (effects (font (size 1.27 1.27)) hide)
-    )
-    (property "Datasheet" "~" (id 3) (at 145.415 86.36 0)
-      (effects (font (size 1.27 1.27)) hide)
-    )
-    (pin "1")
-    (pin "2")
-  )
-  (symbol (lib_id "Linux-capable-PCB-KiCAD-rescue:C-Device") (at 132.715 86.36 0) (unit 1)
-    (in_bom yes) (on_board yes)
-    (property "Reference" "C50" (id 0) (at 135.636 85.1916 0)
-      (effects (font (size 1.27 1.27)) (justify left))
-    )
-    (property "Value" "100n" (id 1) (at 135.636 87.503 0)
-      (effects (font (size 1.27 1.27)) (justify left))
-    )
-    (property "Footprint" "Capacitor_SMD:C_0603_1608Metric" (id 2) (at 133.6802 90.17 0)
-      (effects (font (size 1.27 1.27)) hide)
-    )
-    (property "Datasheet" "~" (id 3) (at 132.715 86.36 0)
-      (effects (font (size 1.27 1.27)) hide)
-    )
-    (pin "1")
-    (pin "2")
-  )
-  (symbol (lib_id "power:GND") (at 132.715 92.71 0) (unit 1)
-    (in_bom yes) (on_board yes)
-    (property "Reference" "#PWR0210" (id 0) (at 132.715 99.06 0)
-      (effects (font (size 1.27 1.27)) hide)
-    )
-    (property "Value" "GND" (id 1) (at 132.842 97.1042 0))
-    (property "Footprint" "" (id 2) (at 132.715 92.71 0)
-      (effects (font (size 1.27 1.27)) hide)
-    )
-    (property "Datasheet" "" (id 3) (at 132.715 92.71 0)
-      (effects (font (size 1.27 1.27)) hide)
-    )
-    (pin "1")
-  )
-  (symbol (lib_id "power:GND") (at 145.415 92.71 0) (unit 1)
-    (in_bom yes) (on_board yes)
-    (property "Reference" "#PWR0211" (id 0) (at 145.415 99.06 0)
-      (effects (font (size 1.27 1.27)) hide)
-    )
-    (property "Value" "GND" (id 1) (at 145.542 97.1042 0))
-    (property "Footprint" "" (id 2) (at 145.415 92.71 0)
-      (effects (font (size 1.27 1.27)) hide)
-    )
-    (property "Datasheet" "" (id 3) (at 145.415 92.71 0)
-      (effects (font (size 1.27 1.27)) hide)
-    )
-    (pin "1")
-  )
-  (symbol (lib_id "power:+1V35") (at 139.7 77.47 0) (unit 1)
-    (in_bom yes) (on_board yes)
-    (property "Reference" "#PWR0212" (id 0) (at 139.7 81.28 0)
-      (effects (font (size 1.27 1.27)) hide)
-    )
-    (property "Value" "+1V35" (id 1) (at 140.081 73.0758 0))
-    (property "Footprint" "" (id 2) (at 139.7 77.47 0)
-      (effects (font (size 1.27 1.27)) hide)
-    )
-    (property "Datasheet" "" (id 3) (at 139.7 77.47 0)
-      (effects (font (size 1.27 1.27)) hide)
-    )
-    (pin "1")
-  )
   (symbol (lib_id "Linux-capable-PCB-KiCAD-rescue:R-Device") (at 81.28 130.175 270) (unit 1)
